File: electronic_design/ethersweep2/ethersweep.kicad_pcb (KiCad board)
At the start: 2 copper layers, 79 x 38 mm, 71 parts, among them J1 AVR-ISP-6, J2 Conn_01x02_Male, J3 Conn_01x04_Female, J4 Conn_01x02_Male, J5 Conn_01x02_Male, J6 HR911105A, J7 Conn_01x06_Female, J8 AVR-ISP-6, J9 Conn_01x06_Male, M1 Stepper_Motor_bipolar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

Commit message: design cleanup
Routing:
- net +3V3: track 232.7 -> 226.8 mm
- net GND: vias 191 -> 190
Other:
- board text added: "MOTOR"
Changed lines of the file:
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@@
   (general
     (thickness 1.6)
-    (drawings 52)
-    (tracks 1206)
+    (drawings 53)
+    (tracks 1200)
     (zones 0)
     (modules 71)
@@
     (descr "Through hole IDC box header, 2x03, 2.54mm pitch, DIN 41651 / IEC 60603-13, double rows, https://docs.google.com/spreadsheets/d/16SsEcesNF15N3Lb4niX7dcUr-NY5_MFPQhobNuNppn4/edit#gid=0")
     (tags "Through hole vertical IDC box header THT 2x03 2.54mm double row")
-    (fp_text reference J1 (at -1.6 4.5) (layer F.SilkS)
+    (fp_text reference J1 (at -5.3 12.3) (layer F.SilkS)
       (effects (font (size 1 1) (thickness 0.15)))
     )
@@
     (tags capacitor)
     (attr smd)
-    (fp_text reference C1 (at 2.75 0) (layer F.SilkS)
+    (fp_text reference C1 (at -2.45 0) (layer F.SilkS)
       (effects (font (size 1 1) (thickness 0.15)))
     )
@@
     (tags capacitor)
     (attr smd)
-    (fp_text reference C19 (at -2.5 0 180) (layer F.SilkS)
+    (fp_text reference C19 (at -3.2 0 270) (layer F.SilkS)
       (effects (font (size 1 1) (thickness 0.15)))
     )
@@
     (tags "Surface mounted pin header SMD 2x02 2.54mm double row")
     (attr smd)
-    (fp_text reference M1 (at 0 -3.6) (layer F.SilkS)
+    (fp_text reference M1 (at -0.5 -9.2) (layer F.SilkS)
       (effects (font (size 1 1) (thickness 0.15)))
     )
@@
     (descr "Through hole straight pin header, 1x06, 2.54mm pitch, single row")
     (tags "Through hole pin header THT 1x06 2.54mm single row")
-    (fp_text reference J9 (at 0 -2.33 90) (layer F.SilkS)
+    (fp_text reference J9 (at -1.6 -5.28 90) (layer F.SilkS)
       (effects (font (size 1 1) (thickness 0.15)))
     )
@@
     (tags capacitor)
     (attr smd)
-    (fp_text reference C2 (at 0 -1.85) (layer F.SilkS)
+    (fp_text reference C2 (at 3.375 -0.1) (layer F.SilkS)
       (effects (font (size 1 1) (thickness 0.15)))
     )
@@
       (net 1 GND))
   )
+  (gr_text MOTOR (at 181 86.1) (layer F.SilkS)
+    (effects (font (size 1.1 1.1) (thickness 0.275)))
+  )
   (gr_poly (pts (xy 139.3 91) (xy 139.2 111) (xy 126.2 111) (xy 126.3 91)) (layer B.SilkS) (width 0.1))
   (gr_text ethersweep (at 193.9 85.3) (layer B.SilkS)
@@
   (via (at 166 105) (size 0.8) (drill 0.4) (layers F.Cu B.Cu) (net 1))
   (via (at 179.5 103.5) (size 0.8) (drill 0.4) (layers F.Cu B.Cu) (net 1))
-  (via (at 182.5 95.5) (size 0.8) (drill 0.4) (layers F.Cu B.Cu) (net 1))
-  (via (at 184 95) (size 0.8) (drill 0.4) (layers F.Cu B.Cu) (net 1))
   (segment (start 184.405 97.3) (end 184.7 97.3) (width 0.2) (layer B.Cu) (net 1))
   (segment (start 184.7 97.3) (end 185 97) (width 0.2) (layer B.Cu) (net 1))
@@
   (via (at 179.8 86) (size 0.8) (drill 0.4) (layers F.Cu B.Cu) (net 1))
   (via (at 177.8 99) (size 0.8) (drill 0.4) (layers F.Cu B.Cu) (net 1))
-  (via (at 178.2 96) (size 0.8) (drill 0.4) (layers F.Cu B.Cu) (net 1))
   (via (at 164.2 100) (size 0.8) (drill 0.4) (layers F.Cu B.Cu) (net 1))
   (via (at 165.4 100.2) (size 0.8) (drill 0.4) (layers F.Cu B.Cu) (net 1))
@@
   (via (at 171.5 107.5) (size 0.8) (drill 0.4) (layers F.Cu B.Cu) (net 1))
   (via (at 169.6 105.5) (size 0.8) (drill 0.4) (layers F.Cu B.Cu) (net 1))
+  (via (at 184.2 95.3) (size 0.8) (drill 0.4) (layers F.Cu B.Cu) (net 1))
+  (via (at 178.3 96) (size 0.8) (drill 0.4) (layers F.Cu B.Cu) (net 1))
   (segment (start 148 85.675) (end 147.175 86.5) (width 0.4) (layer F.Cu) (net 2))
   (segment (start 148 84.4375) (end 148 85.675) (width 0.4) (layer F.Cu) (net 2))
@@
   (segment (start 169.065699 98) (end 168.565699 97.5) (width 0.2) (layer F.Cu) (net 6))
   (segment (start 170.5 98) (end 169.065699 98) (width 0.2) (layer F.Cu) (net 6))
-  (segment (start 182.5 94.5) (end 182.5 94.5) (width 0.2) (layer B.Cu) (net 6))
-  (via (at 182.5 94.5) (size 0.8) (drill 0.4) (layers F.Cu B.Cu) (net 6))
   (segment (start 188.225 95.3) (end 188.225 94.3) (width 0.2) (layer F.Cu) (net 6))
   (segment (start 187.524989 96.000011) (end 188.225 95.3) (width 0.2) (layer F.Cu) (net 6))
   (segment (start 184.000011 96.000011) (end 187.524989 96.000011) (width 0.2) (layer F.Cu) (net 6))
-  (segment (start 182.5 94.5) (end 184.000011 96.000011) (width 0.2) (layer F.Cu) (net 6))
-  (segment (start 182 94) (end 177.75 94) (width 0.2) (layer B.Cu) (net 6))
-  (segment (start 182 94) (end 182.5 94.5) (width 0.2) (layer B.Cu) (net 6))
-  (segment (start 174.25 97.5) (end 173.5 97.5) (width 0.2) (layer B.Cu) (net 6))
-  (segment (start 177.75 94) (end 174.25 97.5) (width 0.2) (layer B.Cu) (net 6))
   (segment (start 173.299999 97.299999) (end 173.5 97.5) (width 0.2) (layer F.Cu) (net 6))
   (segment (start 171.163999 97.299999) (end 173.299999 97.299999) (width 0.2) (layer F.Cu) (net 6))
   (segment (start 170.5 97.963998) (end 171.163999 97.299999) (width 0.2) (layer F.Cu) (net 6))
   (segment (start 170.5 98) (end 170.5 97.963998) (width 0.2) (layer F.Cu) (net 6))
+  (segment (start 184.000011 96.000011) (end 183.700011 96.000011) (width 0.2) (layer F.Cu) (net 6))
+  (segment (start 183.700011 96.000011) (end 182.8 95.1) (width 0.2) (layer F.Cu) (net 6))
+  (segment (start 182.8 95.1) (end 182.8 95.1) (width 0.2) (layer F.Cu) (net 6))
+  (via (at 182.8 95.1) (size 0.8) (drill 0.4) (layers F.Cu B.Cu) (net 6))
+  (segment (start 174.25 97.5) (end 173.5 97.5) (width 0.2) (layer B.Cu) (net 6))
+  (segment (start 177.75 94) (end 174.25 97.5) (width 0.2) (layer B.Cu) (net 6))
+  (segment (start 181.7 94) (end 177.75 94) (width 0.2) (layer B.Cu) (net 6))
+  (segment (start 182.8 95.1) (end 181.7 94) (width 0.2) (layer B.Cu) (net 6))
   (segment (start 192.125 95.3) (end 191 96.425) (width 0.2) (layer F.Cu) (net 7))
   (segment (start 192.125 94.3) (end 192.125 95.3) (width 0.2) (layer F.Cu) (net 7))
@@
   (segment (start 181.5 104.5) (end 176 104.5) (width 1) (layer B.Cu) (net 14))
   (segment (start 176 104.5) (end 173.5 102) (width 1) (layer B.Cu) (net 14))
-  (segment (start 181.9125 92.365334) (end 181.9125 92) (width 0.2) (layer F.Cu) (net 14))
-  (segment (start 181.9125 93.0875) (end 180 95) (width 0.4) (layer F.Cu) (net 14))
-  (segment (start 181.9125 92) (end 181.9125 93.0875) (width 0.4) (layer F.Cu) (net 14))
   (segment (start 177.5 95) (end 174.200001 98.299999) (width 0.4) (layer B.Cu) (net 14))
   (segment (start 180 95) (end 177.5 95) (width 0.4) (layer B.Cu) (net 14))
@@
   (segment (start 174.200001 100.299999) (end 172.5 102) (width 0.4) (layer F.Cu) (net 14))
   (segment (start 174.200001 98.299999) (end 174.200001 100.299999) (width 0.4) (layer F.Cu) (net 14))
-  (segment (start 181.9125 92.728498) (end 181.9125 92) (width 0.4) (layer F.Cu) (net 14))
-  (segment (start 181.9125 92.506756) (end 181.9125 92) (width 0.4) (layer F.Cu) (net 14))
-  (segment (start 184.155008 93.85001) (end 183.255754 93.85001) (width 0.4) (layer F.Cu) (net 14))
-  (segment (start 183.255754 93.85001) (end 181.9125 92.506756) (width 0.4) (layer F.Cu) (net 14))
-  (segment (start 185.804999 95.500001) (end 184.155008 93.85001) (width 0.4) (layer F.Cu) (net 14))
-  (segment (start 186.745001 95.500001) (end 185.804999 95.500001) (width 0.4) (layer F.Cu) (net 14))
-  (segment (start 186.925 95.320002) (end 186.745001 95.500001) (width 0.4) (layer F.Cu) (net 14))
-  (segment (start 186.925 94.3) (end 186.925 95.320002) (width 0.4) (layer F.Cu) (net 14))
-  (segment (start 181.9125 92) (end 181.9125 90) (width 0.4) (layer F.Cu) (net 14))
   (segment (start 172.46 87.5) (end 173.750001 88.790001) (width 0.4) (layer B.Cu) (net 14))
   (segment (start 138.725 97.975) (end 138.725 96.9) (width 0.2) (layer F.Cu) (net 14))
@@
   (segment (start 176.100001 110.899999) (end 176.100001 104.600001) (width 0.4) (layer B.Cu) (net 14))
   (segment (start 175 112) (end 176.100001 110.899999) (width 0.4) (layer B.Cu) (net 14))
+  (segment (start 186.925 95.320002) (end 186.925 94.3) (width 0.4) (layer F.Cu) (net 14))
+  (segment (start 180 95) (end 180.700001 94.299999) (width 0.4) (layer F.Cu) (net 14))
+  (segment (start 186.745001 95.500001) (end 186.925 95.320002) (width 0.4) (layer F.Cu) (net 14))
+  (segment (start 185.804999 95.500001) (end 186.745001 95.500001) (width 0.4) (layer F.Cu) (net 14))
+  (segment (start 184.604997 94.299999) (end 185.804999 95.500001) (width 0.4) (layer F.Cu) (net 14))
+  (segment (start 180.700001 94.299999) (end 184.604997 94.299999) (width 0.4) (layer F.Cu) (net 14))
   (segment (start 137.5 109) (end 137.5 109) (width 0.4) (layer F.Cu) (net 15))
   (via (at 137.5 109) (size 0.8) (drill 0.4) (layers F.Cu B.Cu) (net 15))

Commit message: cleanup
Parts:
- moved J3 0.20 mm to (124.0, 103.8)
Routing:
- net rst: track 69.5 -> 70.4 mm
- net GND: track 92.9 -> 92.8 mm, vias 190 -> 192
Other:
- board text added: "by Neumi 2021-02-10"
- board text added: "vers. 2.0.1"
- board text removed: "VERSION: 2.0.1"
- board text removed: "by Neumi 2021-02-05"
